File: Tachiyon-α.kicad_pcb (KiCad board)
At the start: 2 copper layers, 32 x 47 mm, 31 parts, among them J1 USB_B_Micro, J2 Conn_01x04_Pin, J3 Conn_01x10_Pin, J4 Conn_01x10_Pin, U1 MSPM0C1xxx/L1xxx_20pin, U2 AMS1117-3.3, U3 USBLC6-4SC6, U4 CH340N

Commit message: Modify PCB Design to fix Trace Connection
- Use 0.2mm trace in tight spots near VSSOP20 footprint
- Fix Bottom Silkscreen for better label visibility
- Add Vias for better ground connectivity.

Signed-off-by: u592003sd <sarvadnyasonic@gmail.com>
Routing:
- net GND: track 42.6 -> 43.5 mm, vias 17 -> 18
Changed lines of the file:
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@@
 		(tags "Through hole pin header THT 1x10 2.54mm single row")
 		(property "Reference" "J4"
-			(at 1.29 -2.54 0)
+			(at 0.04 -2.29 0)
 			(layer "F.SilkS")
 			(effects
@@
 	)
 	(gr_text "GND"
-		(at 107.75 81.75 0)
+		(at 106.75 81.75 0)
 		(layer "B.SilkS")
 		(effects
@@
 	)
 	(gr_text "PA6"
-		(at 107.75 89.5 0)
+		(at 106.5 89.5 0)
 		(layer "B.SilkS")
 		(effects
@@
 	)
 	(gr_text "PA0"
-		(at 107.25 74.25 0)
+		(at 106.5 74.25 0)
 		(layer "B.SilkS")
 		(effects
@@
 	)
 	(gr_text "PA2"
-		(at 107.75 84.5 0)
+		(at 106.5 84.5 0)
 		(layer "B.SilkS")
 		(effects
@@
 	)
 	(gr_text "PA4"
-		(at 107.75 86.75 0)
+		(at 106.5 87 0)
 		(layer "B.SilkS")
 		(effects
@@
 	)
 	(segment
-		(start 116.81 58.385)
-		(end 119.385 58.385)
-		(width 0.5)
-		(layer "F.Cu")
-		(net 2)
-	)
-	(segment
 		(start 120.75 89.8)
 		(end 119.55 91)
@@
 	)
 	(segment
+		(start 107.25 74.9)
+		(end 107.25 75.75)
+		(width 0.3)
+		(layer "F.Cu")
+		(net 2)
+	)
+	(segment
 		(start 115.45 84.55)
 		(end 115.45 83.15)
@@
 	(segment
 		(start 116.81 58.385)
+		(end 118.75 58.385)
+		(width 0.5)
+		(layer "F.Cu")
+		(net 2)
+	)
+	(segment
+		(start 116.81 58.385)
 		(end 116.81 63.81)
 		(width 0.5)
@@
 	)
 	(segment
+		(start 107.25 75.75)
+		(end 107.75 76.25)
+		(width 0.3)
+		(layer "F.Cu")
+		(net 2)
+	)
+	(segment
 		(start 111.5 68.5)
 		(end 110.6 68.5)
@@
 	)
 	(via
-		(at 119.385 58.385)
+		(at 118.75 58.385)
 		(size 0.8)
 		(drill 0.4)
@@
 	)
 	(via
+		(at 107.75 76.25)
+		(size 0.8)
+		(drill 0.4)
+		(layers "F.Cu" "B.Cu")
+		(net 2)
+	)
+	(via
 		(at 115.25 84.75)
 		(size 0.8)
@@
 	)
 	(segment
-		(start 115.619014 68.5)
-		(end 115 68.5)
-		(width 0.3)
-		(layer "F.Cu")
-		(net 24)
-	)
-	(segment
-		(start 116.036054 68.498)
-		(end 115.828534 68.498)
-		(width 0.3)
-		(layer "F.Cu")
-		(net 24)
-	)
-	(segment
 		(start 113 84.409999)
 		(end 113 83.848519)
@@
 	)
 	(segment
-		(start 116.751 69.212945)
-		(end 116.036054 68.498)
+		(start 115 68.5)
+		(end 116.038055 68.5)
 		(width 0.3)
 		(layer "F.Cu")
@@
 	)
 	(segment
+		(start 116.038055 68.5)
+		(end 116.751 69.212945)
+		(width 0.3)
+		(layer "F.Cu")
+		(net 24)
+	)
+	(segment
 		(start 124.46 81.28)
 		(end 122.5 79.32)
@@
 	)
 	(segment
-		(start 112.5 83.639999)
-		(end 112.5 77)
-		(width 0.3)
-		(layer "F.Cu")
-		(net 25)
-	)
-	(segment
-		(start 123.1 82.25)
-		(end 123.1 82.85)
-		(width 0.5)
+		(start 115 69)
+		(end 115.829534 69)
+		(width 0.2)
 		(layer "F.Cu")
 		(net 25)
 	)
 	(segment
-		(start 116.25 69.420466)
-		(end 115.828534 68.999)
+		(start 112.5 83.639999)
+		(end 112.5 77)
 		(width 0.3)
 		(layer "F.Cu")
@@
 	)
 	(segment
-		(start 114.5 75)
-		(end 113.25 75)
-		(width 0.3)
+		(start 115.829534 69)
+		(end 116.25 69.420466)
+		(width 0.2)
 		(layer "F.Cu")
 		(net 25)
 	)
 	(segment
-		(start 115.828534 68.999)
-		(end 115.827534 69)
-		(width 0.3)
+		(start 123.1 82.25)
+		(end 123.1 82.85)
+		(width 0.5)
 		(layer "F.Cu")
 		(net 25)
 	)
 	(segment
-		(start 115.827534 69)
-		(end 115 69)
+		(start 114.5 75)
+		(end 113.25 75)
 		(width 0.3)
 		(layer "F.Cu")
