File: Tachiyon-α.kicad_pcb (KiCad board)
At the start: 2 copper layers, 32 x 47 mm, 31 parts, among them J1 USB_B_Micro, J2 Conn_01x04_Pin, J3 Conn_01x10_Pin, J4 Conn_01x10_Pin, U1 MSPM0C1xxx/L1xxx_20pin, U2 AMS1117-3.3, U3 USBLC6-4SC6, U4 CH340N

Commit message: Modify AMS1117 Power Input Filter Stage
- Remove Pi Filter at AMS1117 input stage and
  add a ferrite bead for EMI suppression
- Reduce Input and output stability capacitor value of AMS1117
  from 22uF to 10uF to accomodate USB2.0 bus capacitance requirements
- Modify PCB design to incorporate schematic changes
- Generate gerber files for new PCB Layout

Signed-off-by: u592003sd <sarvadnyasonic@gmail.com>
Parts:
- removed C6: 470nF, Capacitor_SMD:C_0603_1608Metric
- removed R4: 5k1, Resistor_SMD:R_0603_1608Metric
- added FB1: 33R, Resistor_SMD:R_0603_1608Metric, F.Cu at (116.2, 91.8)
- C3, C4: value 22u -> 10u
- C5: value 470nF -> 10nF
Routing:
- net GND: track 43.5 -> 40.6 mm
